File: PCB/make_nn_bot.sch (KiCad schematic (older format))
At the start: 56 parts, among them P1 USB_OTG, P17 DBG_CONN, P2 BatteryHolder, P3 CONN_01X07, P4 MOTOR_A, P5 MOTOR_B, Q1 Q_PMOS_DSG, Q2 Q_PMOS_GSD, SW2 SW_PUSH, SW3 SW_PUSH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

Commit message: small revisions
Parts:
- C1, C11, C12, C3, C5: Digikey Part No. 311-1343-1-ND -> 478-1239-1-ND
- C10, C7: Digikey Part No. 490-5915-1-ND -> 490-5421-1-ND
- C13: Digikey Part No. 311-1729-1-ND -> 587-1256-1-ND
- C14, C15: Digikey Part No. 490-6328-1-ND -> 478-1239-1-ND
- C2, C4: Digikey Part No. 712-1261-1-ND -> 1276-2192-1-ND
- C6: Digikey Part No. 1276-1291-1-ND -> 587-1430-1-ND
- C8: Digikey Part No. 490-1320-1-ND -> 1276-1946-1-ND
- C9: Digikey Part No. 490-10451-1-ND -> 587-1430-1-ND
- P1: symbol USB_OTG -> USB_OTG-RESCUE-make_nn_bot
- P3: Digikey Part No. (none) -> S7040-ND
- R1: Digikey Part No. 311-100KLRCT-ND -> 311-100KHRCT-ND
- R11, R15, R3, R6, R9: Digikey Part No. 311-10KJRCT-ND -> 311-10KGRCT-ND
- R13, R14, R19: Digikey Part No. 311-1.0KJRCT-ND -> 311-1.0KGRCT-ND
- R18: Digikey Part No. 311-33KJRCT-ND -> 311-33KGRCT-ND
- R2: Digikey Part No. 311-330JRCT-ND -> 311-330GRCT-ND
- R4, R5: Digikey Part No. 311-47.0KLRCT-ND -> 311-47.0KHRCT-ND
- SW2: Digikey Part No. CKN9112CT-ND -> 401-1702-1-ND
- SW3: Digikey Part No. CKN9084CT-ND -> 401-1702-1-ND
- Y1: Digikey Part No. 631-1002-1-ND -> XC1617CT-ND
Changed lines of the file:
@@
 EESchema Schematic File Version 2
+LIBS:make_nn_bot-rescue
 LIBS:power
 LIBS:device
@@
 F 2 "Resistors_SMD:R_0603" H 2150 1350 60  0001 C CNN
 F 3 "" H 2150 1350 60  0000 C CNN
-F 4 "311-10KJRCT-ND" H 2150 1350 60  0001 C CNN "Digikey Part No."
+F 4 "311-10KGRCT-ND" H 2150 1350 60  0001 C CNN "Digikey Part No."
 	1    2150 1350
 	1    0    0    -1
@@
 F 2 "Capacitors_SMD:C_0603" H 1650 1950 60  0001 C CNN
 F 3 "" H 1650 1950 60  0000 C CNN
-F 4 "311-1343-1-ND" H 1650 1950 60  0001 C CNN "Digikey Part No."
+F 4 "478-1239-1-ND" H 1650 1950 60  0001 C CNN "Digikey Part No."
 	1    1650 1950
 	1    0    0    -1
@@
 F 2 "Capacitors_SMD:C_0603" H 1800 1950 60  0001 C CNN
 F 3 "" H 1800 1950 60  0000 C CNN
-F 4 "311-1343-1-ND" H 1800 1950 60  0001 C CNN "Digikey Part No."
+F 4 "478-1239-1-ND" H 1800 1950 60  0001 C CNN "Digikey Part No."
 	1    1800 1950
 	1    0    0    -1
@@
 F 2 "Capacitors_SMD:C_0603" H 1100 2450 60  0001 C CNN
 F 3 "" H 1100 2450 60  0000 C CNN
-F 4 "311-1343-1-ND" H 1100 2450 60  0001 C CNN "Digikey Part No."
+F 4 "478-1239-1-ND" H 1100 2450 60  0001 C CNN "Digikey Part No."
 	1    1100 2450
 	1    0    0    -1
@@
 F 2 "Capacitors_SMD:C_0603" H 1250 2850 60  0001 C CNN
 F 3 "" H 1250 2850 60  0000 C CNN
-F 4 "712-1261-1-ND" H 1250 2850 60  0001 C CNN "Digikey Part No."
+F 4 "1276-2192-1-ND" H 1250 2850 60  0001 C CNN "Digikey Part No."
 	1    1250 2850
 	1    0    0    -1
@@
 F 2 "Capacitors_SMD:C_0603" H 1450 2850 60  0001 C CNN
 F 3 "" H 1450 2850 60  0000 C CNN
-F 4 "712-1261-1-ND" H 1450 2850 60  0001 C CNN "Digikey Part No."
+F 4 "1276-2192-1-ND" H 1450 2850 60  0001 C CNN "Digikey Part No."
 	1    1450 2850
 	1    0    0    -1
@@
 F 2 "project_footprints:crystal_smd_5x3.2mm" H 1350 2600 60  0001 C CNN
 F 3 "" H 1350 2600 60  0000 C CNN
-F 4 "631-1002-1-ND" H 1350 2600 60  0001 C CNN "Digikey Part No."
+F 4 "XC1617CT-ND" H 1350 2600 60  0001 C CNN "Digikey Part No."
 	1    1350 2600
 	-1   0    0    1
@@
 F 2 "Capacitors_SMD:C_0603" H 6800 1650 60  0001 C CNN
 F 3 "" H 6800 1650 60  0000 C CNN
-F 4 "311-1343-1-ND" H 6800 1650 60  0001 C CNN "Digikey Part No."
+F 4 "478-1239-1-ND" H 6800 1650 60  0001 C CNN "Digikey Part No."
 	1    6800 1650
 	1    0    0    -1
@@
 F 2 "Capacitors_SMD:C_0603" H 7000 1650 60  0001 C CNN
 F 3 "" H 7000 1650 60  0000 C CNN
-F 4 "311-1343-1-ND" H 7000 1650 60  0001 C CNN "Digikey Part No."
+F 4 "478-1239-1-ND" H 7000 1650 60  0001 C CNN "Digikey Part No."
 	1    7000 1650
 	1    0    0    -1
@@
 $EndComp
 $Comp
-L USB_OTG P1
+L USB_OTG-RESCUE-make_nn_bot P1
 U 1 1 56BE58D4
 P 1550 7850
@@
 F 2 "Capacitors_SMD:C_0603" H 2700 7850 60  0001 C CNN
 F 3 "" H 2700 7850 60  0000 C CNN
-F 4 "1276-1291-1-ND" H 2700 7850 60  0001 C CNN "Digikey Part No."
+F 4 "587-1430-1-ND" H 2700 7850 60  0001 C CNN "Digikey Part No."
 	1    2700 7850
 	1    0    0    -1
@@
 F 2 "Capacitors_SMD:C_0603" H 4250 7900 60  0001 C CNN
 F 3 "" H 4250 7900 60  0000 C CNN
-F 4 "490-1320-1-ND" H 4250 7900 60  0001 C CNN "Digikey Part No."
+F 4 "1276-1946-1-ND" H 4250 7900 60  0001 C CNN "Digikey Part No."
 	1    4250 7900
 	1    0    0    -1
@@
 F 2 "Resistors_SMD:R_0603" H 3800 7850 60  0001 C CNN
 F 3 "" H 3800 7850 60  0000 C CNN
-F 4 "311-47.0KLRCT-ND" H 3800 7850 60  0001 C CNN "Digikey Part No."
+F 4 "311-47.0KHRCT-ND" H 3800 7850 60  0001 C CNN "Digikey Part No."
 	1    3800 7850
 	1    0    0    -1
@@
 F 2 "Resistors_SMD:R_0603" H 1300 8700 60  0001 C CNN
 F 3 "" H 1300 8700 60  0000 C CNN
-F 4 "311-100KLRCT-ND" H 1300 8700 60  0001 C CNN "Digikey Part No."
+F 4 "311-100KHRCT-ND" H 1300 8700 60  0001 C CNN "Digikey Part No."
 	1    1300 8700
 	1    0    0    -1
@@
 F 2 "Resistors_SMD:R_0603" H 1300 9000 60  0001 C CNN
 F 3 "" H 1300 9000 60  0000 C CNN
-F 4 "311-330JRCT-ND" H 1300 9000 60  0001 C CNN "Digikey Part No."
+F 4 "311-330GRCT-ND" H 1300 9000 60  0001 C CNN "Digikey Part No."
 	1    1300 9000
 	1    0    0    -1
@@
 F 2 "Capacitors_SMD:C_0603" H 5700 7900 60  0001 C CNN
 F 3 "" H 5700 7900 60  0000 C CNN
-F 4 "490-10451-1-ND" H 5700 7900 60  0001 C CNN "Digikey Part No."
+F 4 "587-1430-1-ND" H 5700 7900 60  0001 C CNN "Digikey Part No."
 	1    5700 7900
 	1    0    0    -1
@@
 F 2 "Capacitors_SMD:C_0603" H 10300 8250 60  0001 C CNN
 F 3 "" H 10300 8250 60  0000 C CNN
-F 4 "490-6328-1-ND" H 10300 8250 60  0001 C CNN "Digikey Part No."
+F 4 "478-1239-1-ND" H 10300 8250 60  0001 C CNN "Digikey Part No."
 	1    10300 8250
 	1    0    0    -1
@@
 F 2 "Capacitors_SMD:C_0603" H 12250 8250 60  0001 C CNN
 F 3 "" H 12250 8250 60  0000 C CNN
-F 4 "490-6328-1-ND" H 12250 8250 60  0001 C CNN "Digikey Part No."
+F 4 "478-1239-1-ND" H 12250 8250 60  0001 C CNN "Digikey Part No."
 	1    12250 8250
 	1    0    0    -1
@@
 F 2 "Capacitors_SMD:C_0603" H 10050 8250 60  0001 C CNN
 F 3 "" H 10050 8250 60  0000 C CNN
-F 4 "311-1729-1-ND" H 10050 8250 60  0001 C CNN "Digikey Part No."
+F 4 "587-1256-1-ND" H 10050 8250 60  0001 C CNN "Digikey Part No."
 	1    10050 8250
 	1    0    0    -1
@@
 F 2 "Buttons_Switches_SMD:SW_SPST_EVQPE1" H 8850 2500 60  0001 C CNN
 F 3 "" H 8850 2500 60  0000 C CNN
-F 4 "CKN9112CT-ND" H 8850 2500 60  0001 C CNN "Digikey Part No."
+F 4 "401-1702-1-ND" H 8850 2500 60  0001 C CNN "Digikey Part No."
 	1    8850 2500
 	1    0    0    -1
@@
 F 2 "Buttons_Switches_SMD:SW_SPST_EVQPE1" H 8850 2850 60  0001 C CNN
 F 3 "" H 8850 2850 60  0000 C CNN
-F 4 "CKN9084CT-ND" H 8850 2850 60  0001 C CNN "Digikey Part No."
+F 4 "401-1702-1-ND" H 8850 2850 60  0001 C CNN "Digikey Part No."
 	1    8850 2850
 	1    0    0    -1
@@
 F 2 "Resistors_SMD:R_0603" V 8830 3750 30  0001 C CNN
 F 3 "" H 8900 3750 30  0000 C CNN
-F 4 "311-1.0KJRCT-ND" V 8900 3750 60  0001 C CNN "Digikey Part No."
+F 4 "311-1.0KGRCT-ND" V 8900 3750 60  0001 C CNN "Digikey Part No."
 	1    8900 3750
 	-1   0    0    1
@@
 F 2 "Resistors_SMD:R_0603" V 8430 4050 30  0001 C CNN
 F 3 "" H 8500 4050 30  0000 C CNN
-F 4 "311-1.0KJRCT-ND" V 8500 4050 60  0001 C CNN "Digikey Part No."
+F 4 "311-1.0KGRCT-ND" V 8500 4050 60  0001 C CNN "Digikey Part No."
 	1    8500 4050
 	-1   0    0    1
@@
 F 2 "Resistors_SMD:R_0603" V 13830 2150 30  0001 C CNN
 F 3 "" H 13900 2150 30  0000 C CNN
-F 4 "311-10KJRCT-ND" V 13900 2150 60  0001 C CNN "Digikey Part No."
+F 4 "311-10KGRCT-ND" V 13900 2150 60  0001 C CNN "Digikey Part No."
 	1    13900 2150
 	1    0    0    -1
@@
 F 2 "Resistors_SMD:R_0603" H 12750 2000 60  0001 C CNN
 F 3 "" H 12750 2000 60  0000 C CNN
-F 4 "311-47.0KLRCT-ND" H 12750 2000 60  0001 C CNN "Digikey Part No."
+F 4 "311-47.0KHRCT-ND" H 12750 2000 60  0001 C CNN "Digikey Part No."
 	1    12750 2000
 	0    -1   -1   0
@@
 F 2 "Capacitors_SMD:C_0603" H 7050 9500 60  0001 C CNN
 F 3 "" H 7050 9500 60  0000 C CNN
-F 4 "490-5915-1-ND" H 7050 9500 60  0001 C CNN "Digikey Part No."
+F 4 "490-5421-1-ND" H 7050 9500 60  0001 C CNN "Digikey Part No."
 	1    7050 9500
 	1    0    0    -1
@@
 F 2 "Capacitors_SMD:C_0603" H 5450 9450 60  0001 C CNN
 F 3 "" H 5450 9450 60  0000 C CNN
-F 4 "490-5915-1-ND" H 5450 9450 60  0001 C CNN "Digikey Part No."
+F 4 "490-5421-1-ND" H 5450 9450 60  0001 C CNN "Digikey Part No."
 	1    5450 9450
 	1    0    0    -1
@@
 F 2 "Resistors_SMD:R_0603" V 5530 10000 30  0001 C CNN
 F 3 "" H 5600 10000 30  0000 C CNN
-F 4 "311-33KJRCT-ND" V 5600 10000 60  0001 C CNN "Digikey Part No."
+F 4 "311-33KGRCT-ND" V 5600 10000 60  0001 C CNN "Digikey Part No."
 	1    5600 10000
 	-1   0    0    1
@@
 F 2 "Resistors_SMD:R_0603" V 5680 10100 30  0001 C CNN
 F 3 "" H 5750 10100 30  0000 C CNN
-F 4 "311-1.0KJRCT-ND" V 5750 10100 60  0001 C CNN "Digikey Part No."
+F 4 "311-1.0KGRCT-ND" V 5750 10100 60  0001 C CNN "Digikey Part No."
 	1    5750 10100
 	1    0    0    -1
@@
 F 3 "" H 11250 2100 50  0000 C CNN
 F 4 "https://www.aliexpress.com/item/White-0-66-inch-OLED-Display-Module-64x48-0-66-LCD-Screen-SPI-for-Arduino-AVR/32782787258.html?spm=a2g0s.9042311.0.0.qYdk7h" H 11250 2100 60  0001 C CNN "AliExpress"
+F 5 "S7040-ND" H 11250 2100 60  0001 C CNN "Digikey Part No."
 	1    11250 2100
 	1    0    0    -1
@@
 F 2 "Resistors_SMD:R_0603" V 13830 3600 30  0001 C CNN
 F 3 "" H 13900 3600 30  0000 C CNN
-F 4 "311-10KJRCT-ND" V 13900 3600 60  0001 C CNN "Digikey Part No."
+F 4 "311-10KGRCT-ND" V 13900 3600 60  0001 C CNN "Digikey Part No."
 	1    13900 3600
 	1    0    0    -1
@@
 F 2 "Resistors_SMD:R_0603" V 13830 4950 30  0001 C CNN
 F 3 "" H 13900 4950 30  0000 C CNN
-F 4 "311-10KJRCT-ND" V 13900 4950 60  0001 C CNN "Digikey Part No."
+F 4 "311-10KGRCT-ND" V 13900 4950 60  0001 C CNN "Digikey Part No."
 	1    13900 4950
 	1    0    0    -1
@@
 F 2 "Resistors_SMD:R_0603" V 13830 6400 30  0001 C CNN
 F 3 "" H 13900 6400 30  0000 C CNN
-F 4 "311-10KJRCT-ND" V 13900 6400 60  0001 C CNN "Digikey Part No."
+F 4 "311-10KGRCT-ND" V 13900 6400 60  0001 C CNN "Digikey Part No."
 	1    13900 6400
 	1    0    0    -1
